File: pcb/princessPhone.brd (EAGLE design)
At the start: 83.5 x 51.5 mm, 78 parts, among them P1 TC2030-MCP-NL, P2 10118194, P3 95009-7441, Q1 2N7002K, SW1 TL1105, SW2 TL1105, SW3 TL1105, U1 Value, U2 AG1170-S3-VERTICAL, U3 PI32MX170D-PT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

Commit message: Synced package sizes.
Parts:
- C10, C7, C8: device rcl:C0402 -> rcl:C0603
- C5: device rcl:C0805 -> rcl:C0603
- R14, R15, R5, R6, R7: device rcl:R0402 -> rcl:R0603
- moved R7 2.73 mm to (-13.4, -2.44), turned to 270 degrees
- moved R6 2.49 mm to (-15.4, -2.44), turned to 270 degrees
- moved C9 1.16 mm to (-11.9, 18.2)
- moved C7 0.86 mm to (-8.76, -2.51), turned to 90 degrees
- moved C8 0.64 mm to (-7.32, 18.3), turned to 180 degrees
Routing:
- net PIC32_SCL2: track 7.77 -> 6.09 mm
- net PIC32_SDA2: track 5.43 -> 6.74 mm
- net N$4: track 3.46 -> 4.36 mm

Commit message: Post-fab PCB tweaks.
Parts:
- R6, R7: value 10K -> 4.7K
Changed lines of the file:
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@@
 <attribute name="VALUE" x="-12.827" y="-0.635" size="0.0254" layer="27" rot="R270"/>
 </element>
-<element name="R6" library="rcl" package="R0603" value="10K" x="-15.3924" y="-2.4384" smashed="yes" rot="R270">
+<element name="R6" library="rcl" package="R0603" value="4.7K" x="-15.3924" y="-2.4384" smashed="yes" rot="R270">
 <attribute name="NAME" x="-13.3604" y="-1.8034" size="1.27" layer="25" rot="R270"/>
 <attribute name="VALUE" x="-17.4244" y="-1.8034" size="1.27" layer="27" rot="R270"/>
 </element>
-<element name="R7" library="rcl" package="R0603" value="10K" x="-13.4112" y="-2.4384" smashed="yes" rot="R270">
+<element name="R7" library="rcl" package="R0603" value="4.7K" x="-13.4112" y="-2.4384" smashed="yes" rot="R270">
 <attribute name="NAME" x="-11.3792" y="-1.8034" size="1.27" layer="25" rot="R270"/>
 <attribute name="VALUE" x="-15.4432" y="-1.8034" size="1.27" layer="27" rot="R270"/>
